Commit message: fix(simulation): spawn the robot, bridge joint_states, and retract a bad diagnosis
Three of the four things #279 left open turned out to be one real bug, one
already-fixed pair of issues, and one wrong conclusion of mine.

Retracted: "the Camera plugin receives nothing from a topic that is publishing"
was a misdiagnosis. Reproduced away from the simulator (plain rclpy publisher
into dc_bringup) and instrumented camera.cpp: the subscription fires and
collect() sees the image. "Message empty" is measurement.hpp reporting an empty
*Record*, which is exactly what a Camera with detection_modules and no image
saving returns for a frame with no barcode in view -- so both the parked robot
and the blank synthetic frames were legitimately empty. Publishing the demo's own
qrcode_0001 texture produces a full Record with the decoded barcode and an
inspected image on disk. The only defect was the log line itself, which fired
once per poll for a normal condition; it is now throttled and reworded.

Fixed for real:

- /joint_states was permanently silent. waffle.model's JointStatePublisher sets
  <topic>joint_states</topic>, overriding gz-sim's default
  /world/<world>/model/<model>/joint_state; gz advertises that default anyway but
  never publishes on it, and the bridge listened to exactly that. Bridging the
  plugin's own topic also drops this config's dependence on the world and model
  names.
- dc_description's URDF pointed at turtlebot3_gazebo meshes -- the same
  Classic-package-with-no-Jazzy-release problem waffle.model had -- so RViz
  rendered a robot with no geometry.

This also completes #324 and #325, whose acceptance criteria are met by the
duplicate-collision and lidar near-clip fixes already in this branch and verified
here: no collision-name error, gz model --list contains turtlebot3_waffle,
/odom 3.1 Hz + /tf 3.0 Hz + /joint_states 85.8 Hz + /imu 16.3 Hz, a /cmd_vel
round trip moves the robot 0.679 m, /scan gives 360 finite beams over 0.40-11.74 m,
and both cameras give 1280x720 frames with essentially every byte non-zero -- all
headless with no GPU. #324 also asked for progress.txt's #268 entry to be
corrected, since it recorded the collision error as a harmless gz-sim GUI quirk
and asserted the robot spawned without ever checking; that is retracted in place.
New dc_simulation/README.md documents the headless-rendering cost with measured
numbers and the three gz-sim traps this port hit.

Closes #324
Closes #325

Co-Authored-By: Claude Opus 5 <noreply@anthropic.com>
Claude-Session: https://claude.ai/code/session_01Nu4cQFKAHFTg6Y3qLXvyKa
Signed-off-by: David Bensoussan <d.bensoussan@proton.me>

File: dc_description/urdf/turtlebot3_waffle_qrcodes.xacro (robot description, xacro)
@@ -53,5 +53,5 @@
       <origin xyz="-0.064 0 0.0" rpy="0 0 0"/>
       <geometry>
-        <mesh filename="package://turtlebot3_gazebo/models/turtlebot3_common/meshes/waffle_base.dae" scale="0.001 0.001 0.001"/>
+        <mesh filename="package://nav2_minimal_tb3_sim/models/turtlebot3_model/meshes/waffle_base.dae" scale="0.001 0.001 0.001"/>
       </geometry>
       <material name="light_black"/>
@@ -79,5 +79,5 @@
       <origin xyz="0 0 0" rpy="1.57 0 0"/>
       <geometry>
-        <mesh filename="package://turtlebot3_gazebo/models/turtlebot3_common/meshes/tire.dae" scale="0.001 0.001 0.001"/>
+        <mesh filename="package://nav2_minimal_tb3_sim/models/turtlebot3_model/meshes/tire.dae" scale="0.001 0.001 0.001"/>
       </geometry>
       <material name="dark"/>
@@ -105,5 +105,5 @@
       <origin xyz="0 0 0" rpy="1.57 0 0"/>
       <geometry>
-        <mesh filename="package://turtlebot3_gazebo/models/turtlebot3_common/meshes/tire.dae" scale="0.001 0.001 0.001"/>
+        <mesh filename="package://nav2_minimal_tb3_sim/models/turtlebot3_model/meshes/tire.dae" scale="0.001 0.001 0.001"/>
       </geometry>
       <material name="dark"/>
@@ -172,5 +172,5 @@
       <origin xyz="0 0 0" rpy="0 0 0"/>
       <geometry>
-        <mesh filename="package://turtlebot3_gazebo/models/turtlebot3_common/meshes/lds.dae" scale="0.001 0.001 0.001"/>
+        <mesh filename="package://nav2_minimal_tb3_sim/models/turtlebot3_model/meshes/lds.dae" scale="0.001 0.001 0.001"/>
       </geometry>
       <material name="dark"/>

Commit message: fix(demos): aim the QR-code demo's cameras at the codes it stops in front of
The waypoints and the cameras were never related to each other, so the robot
drove the aisles perfectly and read nothing. Three independent errors all push
the code the same way out of frame, and the goal tolerance was never sized
against the lens.

- waffle.model carried a pose on each camera link *and* a pose on the sensor
  inside it. An SDF sensor pose is relative to its parent link, so those add:
  both cameras sat at one point, 133 mm ahead of base_footprint -- which is
  what the waypoints aim -- and 94 mm to its right. dc_description's URDF
  described a third robot again: a 1.300 m ground_base_distance borrowed from a
  taller machine put both cameras 0.6 m underground in TF, and both frame
  joints' -pi/2 was cancelled by the sensor_d455 macro's own +pi/2, so in TF
  they looked straight ahead while the simulated pair looked sideways.
- The 60 goal quaternions were non-unit (norm 1.0126), i.e. headings of 88.6
  and -89.2 degrees rather than +/-90 -- the same transcription error #279
  fixed in the initial pose and left in the goals. The rows sat 25 mm off the
  pallet centres, 0.65 m off the codes in a wide-open aisle, and 50 mm off
  centre in the one with no room to spare.
- yaw_goal_tolerance of 0.2 rad slides the code 0.148 m across the frame at
  aisle 2's 0.73 m standoff, on its own more margin than that aisle has.

Both cameras now sit on the robot's centre line at (0, +/-0.02, 0.539) looking
+/-Y, in the SDF and the URDF alike; the goals are exact +/-90 degrees on the
pallet centres, 0.97 m off the codes in the open aisles and dead centre in the
closed one; and the tolerance is sized against the lens, with the inequality
written out beside it. The AMCL seed pose, hand-placed in RViz and 69 mm out,
becomes the launch file's spawn pose carried through the map/world offset.

Measured with the same ZXing call the Camera measurement makes, teleporting the
robot across the goal-tolerance envelope: 88/135 poses decoded before, 18/45 in
the worst aisle -- including poses Nav2 calls a perfect arrival. After: 72/72 on
the boundary of the envelope where the worst case lives, and 180/180 across all
60 stations, covering all eight codes the world carries. A live pass with the DC
pipeline running read all 20 of aisle 1's codes, one Record per station, with no
navigation failures.

tools/sim/scripts/lint_launch_files.py gains the check that was missing: it
re-derives the readability inequality from the four files that have to agree and
fails on each of the three defects on its own. run.sh gains a `detect` stage that
asserts codes really come back during the waypoint run, wired into ci.yaml's
per-PR sim job. It counts QRCode reads specifically: ZXing's default options try
every symbology, and a run of the stage duly read a "51" off the warehouse
shelving, so a check that accepted any barcode would pass on scenery.

Closes #51

Co-Authored-By: Claude Opus 5 <noreply@anthropic.com>
Claude-Session: https://claude.ai/code/session_018TJPr23iXifRzhjdxujMDT
Signed-off-by: David Bensoussan <d.bensoussan@proton.me>

File: dc_description/urdf/turtlebot3_waffle_qrcodes.xacro (robot description, xacro)
@@ -2,14 +2,37 @@
 <robot name="turtlebot3_waffle"
   xmlns:xacro="http://ros.org/wiki/xacro">
-  <xacro:property name="ground_base_distance" value="1.300"/>
-  <xacro:property name="base_link_x" value="0.0"/>
-  <xacro:property name="base_link_y" value="0.0"/>
-  <xacro:property name="base_link_z" value="${ground_base_distance}"/>
-  <xacro:property name="camera_right_x" value="${0.0 - base_link_x}"/>
-  <xacro:property name="camera_right_y" value="${-0.12 - base_link_y}"/>
-  <xacro:property name="camera_right_z" value="${0.665 - base_link_z}"/>
-  <xacro:property name="camera_left_x" value="${0.0 - base_link_x}"/>
-  <xacro:property name="camera_left_y" value="${0.12 - base_link_y}"/>
-  <xacro:property name="camera_left_z" value="${0.690 - base_link_z}"/>
+  <!-- base_link sits 10 mm above base_footprint (see base_joint below). This used
+       to be a "ground_base_distance" of 1.300 m, borrowed from a much taller
+       robot: every camera offset below is expressed relative to the ground and
+       then rebased onto base_link, so a 1.3 m error put both cameras 0.6 m
+       underground in TF (#51). -->
+  <xacro:property name="base_link_z" value="0.010"/>
+  <!-- Optical centre of each inspection camera, measured from base_footprint.
+       These must match the two rgbd_camera sensors in
+       dc_simulation/worlds/waffle.model: the SDF is what renders the images, this
+       URDF is what publishes camera_{left,right}_depth_optical_frame, and until
+       #51 the two described different cameras: pointing different ways, at
+       different heights, in different places. -->
+  <xacro:property name="camera_x" value="0.0"/>
+  <xacro:property name="camera_y" value="0.02"/>
+  <xacro:property name="camera_z" value="0.539"/>
+  <!-- realsense2_description's sensor_d455 macro does not put the optical origin
+       (camera_*_link) on the frame it is attached to: it offsets it by this much
+       in its own bottom-screw axes. Undo that below so the optical origin lands
+       on camera_{x,y,z} exactly. -->
+  <xacro:property name="d455_offset_x" value="0.01115"/>
+  <xacro:property name="d455_offset_y" value="0.0475"/>
+  <xacro:property name="d455_offset_z" value="0.0145"/>
+  <!-- The sensor_d455 macro is instantiated with a further +pi/2 yaw, so a frame
+       joint of 0 makes a camera look along +Y (the robot's left) and one of pi
+       makes it look along -Y (its right). Both frame joints used to carry -pi/2,
+       which the macro's +pi/2 cancelled: in TF, both cameras looked straight
+       ahead while the simulated pair looked sideways (#51). -->
+  <xacro:property name="camera_left_x" value="${camera_x + d455_offset_y}"/>
+  <xacro:property name="camera_left_y" value="${camera_y - d455_offset_x}"/>
+  <xacro:property name="camera_left_z" value="${camera_z - base_link_z - d455_offset_z}"/>
+  <xacro:property name="camera_right_x" value="${camera_x - d455_offset_y}"/>
+  <xacro:property name="camera_right_y" value="${-camera_y + d455_offset_x}"/>
+  <xacro:property name="camera_right_z" value="${camera_z - base_link_z - d455_offset_z}"/>
   <!-- Init colour -->
   <material name="black">
@@ -195,5 +218,5 @@
     <parent link="base_link"/>
     <child link="camera_right_frame_link"/>
-    <origin xyz="${camera_right_x} ${camera_right_y} ${camera_right_z}" rpy="0 0 ${-pi/2}"/>
+    <origin xyz="${camera_right_x} ${camera_right_y} ${camera_right_z}" rpy="0 0 ${pi}"/>
   </joint>
   <xacro:arg name="use_nominal_extrinsics" default="true"/>
@@ -206,5 +229,5 @@
     <parent link="base_link"/>
     <child link="camera_left_frame_link"/>
-    <origin xyz="${camera_left_x} ${camera_left_y} ${camera_left_z}" rpy="0 0 ${-pi/2}"/>
+    <origin xyz="${camera_left_x} ${camera_left_y} ${camera_left_z}" rpy="0 0 0"/>
   </joint>
   <xacro:arg name="use_nominal_extrinsics" default="true"/>
